Commit message: update

File: xacro/robot2/trackbot.urdf.xacro (robot description, xacro)
@@ -1,7 +1,8 @@
 <?xml version="1.0"?>
-<robot xmlns:xacro="http://www.ros.org/wiki/xacro" name="cartbot">
+<robot xmlns:xacro="http://www.ros.org/wiki/xacro" name="trackbot">
+    <xacro:include filename="$(find cartbot)/xacro/robot2/trackbot.gazebo.xacro" />
     <xacro:property name="body_mass" value="15"/>
     <xacro:property name="body_width" value="0.4"/>
-    <xacro:property name="body_height" value="0.25"/>
+    <xacro:property name="body_height" value="0.5"/>
     <xacro:property name="body_length" value="0.6"/>
     <xacro:property name="wheel_gap" value="0.46"/>
@@ -10,4 +11,10 @@
     <xacro:property name="wheel_width" value="0.04"/>
     <xacro:property name="ground_clearnace" value="0.15"/>
+    <material name="red">
+        <color rgba="1.0 0 0.0 0.8"/>
+    </material>
+    <material name="white">
+        <color rgba="1 1 1 1"/>
+    </material>
     <xacro:macro name="box_inertia" params="m w h d">
         <inertial>
@@ -22,19 +29,26 @@
         </inertial>
     </xacro:macro>
-    <link name="body_link">
+    <link name='base_footprint2'/>
+    <joint name="base_joint2" type="fixed">
+        <parent link="base_footprint2"/>
+        <child link="body_link2"/>
+        <origin xyz="0.0 0.0 ${body_height/2 + ground_clearnace}" rpy="0 0 0"/>
+    </joint>
+    <link name='body_link2'>
         <xacro:box_inertia m="${body_mass}" w="${body_width}" h="${body_height}" d="${body_length}"/>
         <visual>
             <origin xyz="0.0 0.0 0.0" rpy="0.0 0.0 0.0"/>
             <geometry>
-                <box size="${body_width} ${body_height} ${body_length}"/>
+                <box size="${body_length} ${body_width} ${body_height}"/>
             </geometry>
+            <material name="red"/>
         </visual>
         <collision>
             <geometry>
-                <box size="${body_width} ${body_height} ${body_length}"/>
+                <box size="${body_length} ${body_width} ${body_height}"/>
             </geometry>
         </collision>
     </link>
-    <link name="wheel_left_link">
+    <link name='wheel_left_link2'>
         <xacro:cylinder_inertia m="${wheel_mass}" r="${wheel_radius}" h="${wheel_width}"/>
         <visual>
@@ -43,4 +57,5 @@
                 <cylinder length="${wheel_width}" radius="${wheel_radius}"/>
             </geometry>
+            <material name="white"/>
         </visual>
         <collision>
@@ -50,10 +65,13 @@
         </collision>
     </link>
-    <joint name="wheel_left_joint" type="continuous">
-        <parent link="body_link"/>
-        <child link="wheel_left_link"/>
-        <origin xyz="${body_length/2} ${wheel_gap/2 *-1} 0.0" rpy="0.0 ${pi/2} ${pi/2}"/>
+    <joint name="wheel_left_joint2" type="continuous">
+        <parent link="body_link2"/>
+        <child link="wheel_left_link2"/>
+        <origin xyz="-${body_length/2 - wheel_radius} ${wheel_gap/2*1} -${ground_clearnace+body_height/2 - wheel_radius}" rpy="-${pi/2} 0.0 0.0"/>
+        <axis xyz="0 0 1"/>
+        <limit effort="10000" velocity="1000"/>
+        <dynamics damping="1.0" friction="1.0"/>
     </joint>
-    <link name="wheel_right_link">
+    <link name='wheel_right_link2'>
         <xacro:cylinder_inertia m="${wheel_mass}" r="${wheel_radius}" h="${wheel_width}"/>
         <visual>
@@ -62,4 +80,5 @@
                 <cylinder length="${wheel_width}" radius="${wheel_radius}"/>
             </geometry>
+            <material name="white"/>
         </visual>
         <collision>
@@ -69,21 +88,30 @@
         </collision>
     </link>
-    <joint name="wheel_right_joint" type="continuous">
-        <parent link="body_link"/>
-        <child link="wheel_right_link"/>
-        <origin xyz="${body_length/2} ${wheel_gap/2} 0.0" rpy="0.0 ${pi/2} ${pi/2}"/>
+    <joint name="wheel_right_joint2" type="continuous">
+        <parent link="body_link2"/>
+        <child link="wheel_right_link2"/>
+        <origin xyz="-${body_length/2 - wheel_radius} ${wheel_gap/2*-1} -${ground_clearnace+body_height/2 - wheel_radius}" rpy="${pi/2} 0.0 0.0"/>
+        <axis xyz="0 0 -1"/>
+        <limit effort="10000" velocity="1000"/>
+        <dynamics damping="1.0" friction="1.0"/>
     </joint>
-    <joint name="caster_joint" type="continuous">
-        <parent link="body_link"/>
-        <child link="caster_wheel_link"/>
-        <origin xyz="-0.2 0.0 -0.04" rpy="0.0 0.0 0.0" />
+    <joint name="caster_joint2" type="fixed">
+        <parent link="body_link2"/>
+        <child link="caster_wheel_link2"/>
+        <origin xyz="0.2 0.0 -${body_height/2 + ground_clearnace/2}" rpy="0.0 0.0 0.0" />
     </joint>
-    <link name="caster_wheel_link">
+    <link name='caster_wheel_link2'>
         <visual>
             <origin xyz="0.0 0.0 0.0" rpy="0.0 0.0 0.0"/>
             <geometry>
-                <sphere radius="0.065" />
+                <sphere radius="${ground_clearnace/2}" />
             </geometry>
+            <material name="white"/>
         </visual>
+        <collision>
+            <geometry>
+                <sphere radius="${ground_clearnace/2}" />
+            </geometry>
+        </collision>
     </link>
 </robot>
